File: IoT_Module/projekt.brd (EAGLE design)
At the start: 82 x 84 mm, 20 parts, among them IC1 ESP12E_DEVKIT, IC2 LF50CP, IC3 LEVEL_SHIFTER, IC4 LEVEL_SHIFTER, J1 PSH02-02W

Commit message: Added door sensor
Parts:
- removed R5: 470, rcl:R1206
Connections:
- removed net N$4: R5.1, S2.3, S2.4
- net RST: now also S2.3, S2.4; no longer R5.2
Routing:
- net RST: track 101.6 -> 130.4 mm
- net N$4: track 17.8 -> 0.00 mm
Changed lines of the file:
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@@
 <element name="R3" library="rcl" package="R1206" value="56k 1%" x="60.96" y="77.47" rot="R270"/>
 <element name="R4" library="rcl" package="R1206" value="110k 1%" x="64.77" y="40.64" rot="R270"/>
-<element name="R5" library="rcl" package="R1206" value="470" x="41.91" y="34.29" rot="R90"/>
 <element name="S1" library="switch-dil" package="DIP02YL" value="" x="57.15" y="8.89" rot="R90">
 <attribute name="OC_NEWARK" value="unknown" x="57.15" y="8.89" size="1.778" layer="27" rot="R90" display="off"/>
@@
 <wire x1="22.5425" y1="69.215" x2="23.8125" y2="67.31" width="0.6096" layer="16"/>
 </signal>
-<signal name="N$4">
-<contactref element="S2" pad="3"/>
-<contactref element="R5" pad="1"/>
-<contactref element="S2" pad="4"/>
-<wire x1="37.39" y1="24.42" x2="43.89" y2="24.42" width="0.6096" layer="16"/>
-<wire x1="43.89" y1="24.42" x2="40.64" y2="27.67" width="0.6096" layer="1"/>
-<wire x1="40.64" y1="27.67" x2="40.64" y2="33.02" width="0.6096" layer="1"/>
-<wire x1="40.64" y1="33.02" x2="40.792" y2="32.868" width="0.4064" layer="1"/>
-<wire x1="40.792" y1="32.868" x2="41.91" y2="32.868" width="0.4064" layer="1"/>
-</signal>
 <signal name="3.3V">
 <contactref element="IC1" pad="3V3@0"/>
@@
 <signal name="RST">
 <contactref element="IC1" pad="RST"/>
-<contactref element="R5" pad="2"/>
 <contactref element="PL1" pad="11"/>
 <wire x1="33.147" y1="69.0372" x2="33.147" y2="71.0946" width="0.6096" layer="1"/>
@@
 <wire x1="40.0431" y1="59.1185" x2="40.0431" y2="63.0936" width="0.6096" layer="1"/>
 <wire x1="40.0431" y1="49.276" x2="40.0431" y2="59.1185" width="0.6096" layer="16"/>
-<wire x1="40.0431" y1="37.9984" x2="40.0431" y2="49.276" width="0.6096" layer="1"/>
-<wire x1="41.8338" y1="35.8902" x2="40.0431" y2="37.9984" width="0.6096" layer="1"/>
 <wire x1="33.147" y1="71.0946" x2="33.02" y2="71.12" width="0.254" layer="1"/>
-<wire x1="41.8338" y1="35.8902" x2="41.91" y2="35.712" width="0.254" layer="1"/>
 <via x="40.0431" y="59.1185" extent="1-16" drill="0.6096" diameter="1.4224" shape="square"/>
 <via x="40.0431" y="49.276" extent="1-16" drill="0.6096" diameter="1.4224" shape="square"/>
@@
 <wire x1="65.405" y1="56.515" x2="65.405" y2="72.39" width="0.6096" layer="16"/>
 <wire x1="59.055" y1="56.515" x2="65.405" y2="56.515" width="0.6096" layer="16"/>
-<wire x1="52.705" y1="48.895" x2="59.055" y2="56.515" width="0.6096" layer="1"/>
-<wire x1="52.705" y1="36.83" x2="52.705" y2="48.895" width="0.6096" layer="1"/>
-<wire x1="50.8" y1="34.925" x2="52.705" y2="36.83" width="0.6096" layer="1"/>
-<wire x1="41.91" y1="34.925" x2="50.8" y2="34.925" width="0.6096" layer="1"/>
-<wire x1="41.91" y1="35.712" x2="41.91" y2="34.925" width="0.254" layer="1"/>
 <via x="59.055" y="56.515" extent="1-16" drill="0.6096" diameter="1.4224" shape="square"/>
+<contactref element="S2" pad="3"/>
+<contactref element="S2" pad="4"/>
+<wire x1="37.39" y1="24.42" x2="43.89" y2="24.42" width="0.6096" layer="16"/>
+<wire x1="40.0431" y1="49.276" x2="40.0685" y2="49.276" width="0.6096" layer="1"/>
+<wire x1="40.0685" y1="49.276" x2="40.0685" y2="32.1945" width="0.6096" layer="1"/>
+<wire x1="40.0685" y1="32.1945" x2="55.5625" y2="32.1945" width="0.6096" layer="1"/>
+<wire x1="55.5625" y1="32.1945" x2="55.5625" y2="56.388" width="0.6096" layer="1"/>
+<wire x1="55.5625" y1="56.388" x2="59.055" y2="56.388" width="0.6096" layer="1"/>
+<wire x1="59.055" y1="56.388" x2="59.055" y2="56.515" width="0.6096" layer="1"/>
+<wire x1="37.39" y1="24.42" x2="40.0685" y2="24.42" width="0.6096" layer="1"/>
+<wire x1="40.0685" y1="24.42" x2="40.0685" y2="32.1945" width="0.6096" layer="1"/>
 </signal>
 <signal name="D0">
