File: RobotDriver/robotdriver.sch (EAGLE design)
At the start: 8 parts

Commit message: Update
Parts:
- added IC1: LM3940, v-reg:78XXS
Changed lines of the file:
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@@
 <part name="U$4" library="diy-modules" deviceset="ULTRASONIC-HC-SR04" device="#V"/>
 <part name="U$5" library="diy-modules" deviceset="ULTRASONIC-HC-SR04" device="#V"/>
+<part name="IC1" library="v-reg" library_urn="urn:adsk.eagle:library:409" deviceset="78XXS" device="" package3d_urn="urn:adsk.eagle:package:30342/1" value="LM3940"/>
 </parts>
 <sheets>
@@
 <instance part="U$4" gate="G$1" x="162.56" y="109.22"/>
 <instance part="U$5" gate="G$1" x="220.98" y="109.22"/>
+<instance part="IC1" gate="1" x="71.12" y="83.82"/>
 </instances>
 <busses>
@@
 </schematic>
 </drawing>
+<compatibility>
+<note version="8.2" severity="warning">
+Since Version 8.2, EAGLE supports online libraries. The ids
+of those online libraries will not be understood (or retained)
+with this version.
+</note>
+<note version="8.3" severity="warning">
+Since Version 8.3, EAGLE supports URNs for individual library
+assets (packages, symbols, and devices). The URNs of those assets
+will not be understood (or retained) with this version.
+</note>
+<note version="8.3" severity="warning">
+Since Version 8.3, EAGLE supports the association of 3D packages
+with devices in libraries, schematics, and board files. Those 3D
+packages will not be understood (or retained) with this version.
+</note>
+</compatibility>
 </eagle>
